Commit message: 346346346

File: isaac_ros-dev/src/agv_car_gazebo/urdf/car1.urdf (robot description, URDF)
Before this commit: robot new_car, 8 links, 7 joints
Links:
- removed link front_left_steering_wheel_link
- removed link front_right_steering_wheel_link
- added link front_left_wheel_steering_link, mass 0.5; collision cylinder length=0.1 radius=0.03; visual cylinder length=0.1 radius=0.03
- added link front_right_wheel_steering_link, mass 0.5; collision cylinder length=0.1 radius=0.03; visual cylinder length=0.1 radius=0.03
Joints:
- joint front_left_wheel_joint: parent front_left_steering_wheel_link -> front_left_wheel_steering_link
- joint front_left_wheel_steering_joint: child front_left_steering_wheel_link -> front_left_wheel_steering_link
- joint front_right_wheel_joint: parent front_right_steering_wheel_link -> front_right_wheel_steering_link
- joint front_right_wheel_steering_joint: child front_right_steering_wheel_link -> front_right_wheel_steering_link
