Commit message: ackermann steering

File: isaac_ros-dev/src/agv_car_gazebo/urdf/car.xacro (robot description, xacro)
@@ -132,4 +132,79 @@
     </joint>
   </xacro:macro>
+  <!-- <link name="velodyne">
+  <visual>
+    <origin rpy="0 0 0" xyz="0 0 0"/>
+    <geometry>
+      <cylinder length=".0762" radius=".0762"/>
+    </geometry>
+    <material name="Cyan">
+      <color rgba="0 1.0 1.0 1.0"/>
+    </material>
+  </visual>
+    <gazebo>
+      <sensor type="gpu_ray" name="velodyne_lidar">
+        <pose>0 0 0 0 0 0</pose>
+        <visualize>true</visualize>
+        <update_rate>20</update_rate>
+        <ray>
+          <scan>
+            <horizontal>
+              <samples>720</samples>
+              <resolution>1</resolution>
+              <min_angle>-1.5708</min_angle>
+              <max_angle>1.5708</max_angle>
+            </horizontal>
+          </scan>
+          <range>
+            <min>0.1</min>
+            <max>30.0</max>
+            <resolution>0.01</resolution>
+          </range>
+        </ray>
+        <plugin name="gazebo_ros_laser" filename="libgazebo_ros_laser.so">
+          <topicName>/scan</topicName>
+          <frameName>velodyne</frameName>
+        </plugin>
+      </sensor>
+    </gazebo>
+  </link>
+  <joint name="velodyne_joint" type="fixed">
+    <parent link="base_link"/>
+    <child link="velodyne"/>
+    <origin xyz ="0 0 1.0414" rpy="0 0 0"/>
+  </joint>
+   <joint name="imu_joint" type="fixed">
+    <parent link="base_link"/>
+    <child link="imu_link"/>
+    <origin xyz="0.0 0 0.068" rpy="0 0 0"/>
+  </joint>
+  <link name="imu_link"/>
+  <joint name="scan_joint" type="fixed">
+    <parent link="base_link"/>
+    <child link="base_scan"/>
+    <origin xyz="-0.064 0 0.122" rpy="0 0 0"/>
+  </joint>
+  <link name="base_scan">
+    <visual>
+      <origin xyz=".946 .521 -.313" rpy="0 0 ${pi}"/>
+      <geometry>
+        <mesh filename="package://agv_car_gazebo/models/agv_car/meshes/agv_chassis.stl"/>
+      </geometry>
+      <material name="dark"/>
+    </visual>
+    <collision>
+      <origin xyz="0.015 0 -0.0065" rpy="0 0 0"/>
+      <geometry>
+        <cylinder length="0.0315" radius="0.055"/>
+      </geometry>
+    </collision>
+    <inertial>
+      <mass value="0.114" />
+      <origin xyz="0 0 0" />
+      <inertia ixx="0.001" ixy="0.0" ixz="0.0"
+               iyy="0.001" iyz="0.0"
+               izz="0.001" />
+    </inertial>
+  </link> -->
   <xacro:rearwheel prefix="left" x_reflect="-1" y_reflect="1" />
   <xacro:rearwheel prefix="right" x_reflect="-1" y_reflect="-1" />

Commit message: test

File: isaac_ros-dev/src/agv_car_gazebo/urdf/car.xacro (robot description, xacro)
@@ -132,4 +132,20 @@
     </joint>
   </xacro:macro>
+    <!-- Ackermann Steering Plugin -->
+  <plugin filename="gz-sim-ackermann-steering" name="gz::sim::systems::AckermannSteering">
+      <left_joint>rear_left_wheel_joint</left_joint>
+      <right_joint>rear_right_wheel_joint</right_joint>
+      <front_left_joint>front_left_steering_joint</front_left_joint>
+      <front_right_joint>front_right_steering_joint</front_right_joint>
+      <wheel_separation>0.287</wheel_separation>
+      <wheel_radius>${wheel_radius}</wheel_radius>
+      <max_linear_acceleration>0.033</max_linear_acceleration>
+      <topic>cmd_vel</topic>
+      <odom_topic>odom</odom_topic>
+      <frame_id>odom</frame_id>
+      <child_frame_id>base_footprint</child_frame_id>
+      <odom_publisher_frequency>30</odom_publisher_frequency>
+      <tf_topic>/tf</tf_topic>
+  </plugin>
   <!-- <link name="velodyne">
   <visual>

File: isaac_ros-dev/src/agv_car_gazebo/urdf/car1.urdf (robot description, URDF)
Before this commit: robot new_car, 8 links, 7 joints
Links:
- removed link front_left_steering_wheel_link
- removed link front_left_wheel
- removed link front_right_steering_wheel_link
- removed link front_right_wheel
- added link front_left_steering_wheel, mass 0.5; collision cylinder length=0.1 radius=0.03; visual cylinder length=0.1 radius=0.03
- added link front_right_steering_wheel, mass 0.5; collision cylinder length=0.1 radius=0.03; visual cylinder length=0.1 radius=0.03
Joints:
- removed joint front_left_wheel_joint
- removed joint front_left_wheel_steering_joint
- removed joint front_right_wheel_joint
- removed joint front_right_wheel_steering_joint
- added joint front_left_steering_joint: type revolute, parent base_link, child front_left_steering_wheel, origin xyz=0.756 0.46049999999999996 -0.123 rpy=0 0 0, axis 0 0 1, limit lower=-0.698 upper=0.698 effort=1000.0 velocity=0.5
- added joint front_right_steering_joint: type revolute, parent base_link, child front_right_steering_wheel, origin xyz=0.756 -0.46049999999999996 -0.123 rpy=0 0 0, axis 0 0 1, limit lower=-0.698 upper=0.698 effort=1000.0 velocity=0.5

Commit message: Test

File: isaac_ros-dev/src/agv_car_gazebo/urdf/car.xacro (robot description, xacro)
@@ -26,20 +26,37 @@
   <!-- Robot Base -->
   <link name="base_link">
-    <visual>
-      <origin xyz=".946 .521 -.313" rpy="0 0 ${pi}" />
-        <geometry>
-        <!-- <box size="${base_length} ${base_width} ${base_height}"/> -->
-          <mesh filename="package://agv_car_gazebo/models/agv_car/meshes/agv_chassis.stl"/>
-        </geometry>
-        <material name="Cyan">
-        <color rgba="0 1.0 1.0 1.0"/>
-        </material>
-    </visual>
-    <collision>
-      <geometry>
-        <mesh filename="package://agv_car_gazebo/models/agv_car/meshes/agv_chassis.stl"/>
-      </geometry>
-    </collision>
-    <xacro:box_inertia m="15" w="${base_width}" d="${base_length}" h="${base_height}"/>
+      <visual>
+          <origin xyz=".946 .521 -.313" rpy="0 0 ${pi}" />
+          <geometry>
+              <mesh filename="package://agv_car_gazebo/models/agv_car/meshes/agv_chassis.stl"/>
+          </geometry>
+          <material name="Cyan">
+              <color rgba="0 1.0 1.0 1.0"/>
+          </material>
+      </visual>
+      <collision>
+          <geometry>
+              <mesh filename="package://agv_car_gazebo/models/agv_car/meshes/agv_chassis.stl"/>
+          </geometry>
+      </collision>
+      <xacro:box_inertia m="15" w="${base_width}" d="${base_length}" h="${base_height}"/>
+      <!-- Ackermann Steering Plugin -->
+      <gazebo>
+          <plugin filename="libgz-sim-ackermann-steering.so" name="gz::sim::systems::AckermannSteering">
+              <left_joint>rear_left_wheel_joint</left_joint>
+              <right_joint>rear_right_wheel_joint</right_joint>
+              <front_left_joint>front_left_wheel_steering_joint</front_left_joint>
+              <front_right_joint>front_right_wheel_steering_joint</front_right_joint>
+              <wheel_separation>0.287</wheel_separation>
+              <wheel_radius>${wheel_radius}</wheel_radius>
+              <max_linear_acceleration>0.033</max_linear_acceleration>
+              <topic>cmd_vel</topic>
+              <odom_topic>odom</odom_topic>
+              <frame_id>odom</frame_id>
+              <child_frame_id>base_footprint</child_frame_id>
+              <odom_publisher_frequency>30</odom_publisher_frequency>
+              <tf_topic>/tf</tf_topic>
+          </plugin>
+      </gazebo>
   </link>
   <!-- Robot Footprint -->
@@ -105,5 +122,5 @@
     </joint>
   </xacro:macro>
-<xacro:macro name="frontwheel" params="prefix x_reflect y_reflect">
+  <xacro:macro name="frontwheel" params="prefix x_reflect y_reflect">
     <link name="front_${prefix}_wheel">
       <visual>
@@ -132,20 +149,4 @@
     </joint>
   </xacro:macro>
-    <!-- Ackermann Steering Plugin -->
-  <plugin filename="gz-sim-ackermann-steering" name="gz::sim::systems::AckermannSteering">
-      <left_joint>rear_left_wheel_joint</left_joint>
-      <right_joint>rear_right_wheel_joint</right_joint>
-      <front_left_joint>front_left_steering_joint</front_left_joint>
-      <front_right_joint>front_right_steering_joint</front_right_joint>
-      <wheel_separation>0.287</wheel_separation>
-      <wheel_radius>${wheel_radius}</wheel_radius>
-      <max_linear_acceleration>0.033</max_linear_acceleration>
-      <topic>cmd_vel</topic>
-      <odom_topic>odom</odom_topic>
-      <frame_id>odom</frame_id>
-      <child_frame_id>base_footprint</child_frame_id>
-      <odom_publisher_frequency>30</odom_publisher_frequency>
-      <tf_topic>/tf</tf_topic>
-  </plugin>
   <!-- <link name="velodyne">
   <visual>

File: isaac_ros-dev/src/agv_car_gazebo/urdf/cartest.xacro (robot description, xacro)
@@ -10,11 +10,10 @@
     <xacro:property name="wheel_zoff" value="0.123"/>
     <xacro:property name="wheel_xoff" value="0.756"/>
-    <!-- Inertia Macros -->
+    <!-- Inertial Macros -->
     <xacro:macro name="box_inertia" params="m w h d">
         <inertial>
             <origin xyz="0 0 0" rpy="${pi/2} 0 ${pi/2}"/>
             <mass value="${m}"/>
-            <inertia ixx="${(m/12) * (h*h + d*d)}" ixy="0.0" ixz="0.0"
-                     iyy="${(m/12) * (w*w + d*d)}" iyz="0.0" izz="${(m/12) * (w*w + h*h)}"/>
+            <inertia ixx="${(m/12) * (h*h + d*d)}" ixy="0.0" ixz="0.0" iyy="${(m/12) * (w*w + d*d)}" iyz="0.0" izz="${(m/12) * (w*w + h*h)}"/>
         </inertial>
     </xacro:macro>
@@ -23,6 +22,5 @@
             <origin xyz="0 0 0" rpy="${pi/2} 0 0"/>
             <mass value="${m}"/>
-            <inertia ixx="${(m/12) * (3*r*r + h*h)}" ixy="0" ixz="0"
-                     iyy="${(m/12) * (3*r*r + h*h)}" iyz="0" izz="${(m/2) * (r*r)}"/>
+            <inertia ixx="${(m/12) * (3*r*r + h*h)}" ixy="0" ixz="0" iyy="${(m/12) * (3*r*r + h*h)}" iyz="0" izz="${(m/2) * (r*r)}"/>
         </inertial>
     </xacro:macro>
@@ -45,4 +43,5 @@
         <xacro:box_inertia m="15" w="${base_width}" d="${base_length}" h="${base_height}"/>
     </link>
+    <!-- Robot Footprint -->
     <link name="base_footprint"/>
     <joint name="base_joint" type="fixed">
@@ -51,7 +50,7 @@
         <origin xyz="0.0 0.0 ${-(wheel_radius + wheel_zoff)}" rpy="0 0 0"/>
     </joint>
-    <!-- Wheel Macro -->
-    <xacro:macro name="wheel" params="prefix x_reflect y_reflect">
-        <link name="${prefix}_wheel">
+    <!-- Wheels -->
+    <xacro:macro name="rearwheel" params="prefix x_reflect y_reflect">
+        <link name="rear_${prefix}_wheel">
             <visual>
                 <origin xyz="0 0 0" rpy="${pi/2} 0 0"/>
@@ -71,17 +70,16 @@
             <xacro:cylinder_inertia m="0.5" r="${wheel_radius}" h="${wheel_width}"/>
         </link>
-        <joint name="${prefix}_wheel_joint" type="revolute">
+        <joint name="rear_${prefix}_wheel_joint" type="revolute">
             <parent link="base_link"/>
-            <child link="${prefix}_wheel"/>
-            <origin xyz="${x_reflect * wheel_xoff} ${y_reflect * (base_width/2 + wheel_ygap)} ${-wheel_zoff}" rpy="0 0 0"/>
+            <child link="rear_${prefix}_wheel"/>
+            <origin xyz="${x_reflect * wheel_xoff} ${y_reflect * (base_width / 2 + wheel_ygap)} ${-wheel_zoff}" rpy="0 0 0"/>
             <axis xyz="0 0 1"/>
             <limit effort="1000.0" lower="-0.698" upper="0.698" velocity="0.5"/>
         </joint>
     </xacro:macro>
-    <!-- Steering Wheel Macro -->
     <xacro:macro name="steering_wheel" params="prefix x_reflect y_reflect">
-        <link name="${prefix}_steering_wheel">
+        <link name="front_${prefix}_wheel_steering_link">
             <visual>
-                <origin xyz="0.05 ${y_reflect * (wheel_width / 2 - .1)} 0" rpy="${pi/2} ${pi/2} 0"/>
+                <origin xyz="0.05 ${y_reflect * (wheel_width / 2 - 0.1)} 0" rpy="${pi/2} ${pi/2} 0"/>
                 <geometry>
                     <cylinder radius="0.03" length="0.1"/>
@@ -92,14 +90,14 @@
             </visual>
             <collision>
-                <origin xyz="0 0 0" rpy="0 -0 0"/>
+                <origin xyz="0 0 0" rpy="0 0 0"/>
                 <geometry>
                     <cylinder radius="0.03" length="0.1"/>
                 </geometry>
             </collision>
-            <xacro:cylinder_inertia m="0.5" r="0.03" h="0.1"/>
+            <xacro:cylinder_inertia m="0.5" r="${wheel_radius}" h="${wheel_width}"/>
         </link>
-        <joint name="${prefix}_steering_joint" type="revolute">
+        <joint name="front_${prefix}_wheel_steering_joint" type="revolute">
             <parent link="base_link"/>
-            <child link="${prefix}_steering_wheel"/>
+            <child link="front_${prefix}_wheel_steering_link"/>
             <origin xyz="${x_reflect * wheel_xoff} ${y_reflect * (base_width / 2 + wheel_ygap)} ${-wheel_zoff}" rpy="0 0 0"/>
             <axis xyz="0 0 1"/>
@@ -107,24 +105,64 @@
         </joint>
     </xacro:macro>
-    <!-- Front and Rear Wheels -->
-    <xacro:wheel prefix="rear_left" x_reflect="-1" y_reflect="1"/>
-    <xacro:wheel prefix="rear_right" x_reflect="-1" y_reflect="-1"/>
-    <xacro:steering_wheel prefix="front_left" x_reflect="1" y_reflect="1"/>
-    <xacro:steering_wheel prefix="front_right" x_reflect="1" y_reflect="-1"/>
+    <xacro:macro name="frontwheel" params="prefix x_reflect y_reflect">
+        <link name="front_${prefix}_wheel">
+            <visual>
+                <origin xyz="0 0 0" rpy="${pi/2} 0 0"/>
+                <geometry>
+                    <cylinder radius="${wheel_radius}" length="${wheel_width}"/>
+                </geometry>
+                <material name="Gray">
+                    <color rgba="0.5 0.5 0.5 1.0"/>
+                </material>
+            </visual>
+            <collision>
+                <origin xyz="0 0 0" rpy="${pi/2} 0 0"/>
+                <geometry>
+                    <cylinder radius="${wheel_radius}" length="${wheel_width}"/>
+                </geometry>
+            </collision>
+            <xacro:cylinder_inertia m="0.5" r="${wheel_radius}" h="${wheel_width}"/>
+        </link>
+        <joint name="front_${prefix}_wheel_joint" type="revolute">
+            <parent link="front_${prefix}_wheel_steering_link"/>
+            <child link="front_${prefix}_wheel"/>
+            <origin xyz="0 0 0" rpy="0 0 0"/>
+            <axis xyz="0 0 1"/>
+            <limit effort="1000.0" lower="-0.698" upper="0.698" velocity="0.5"/>
+        </joint>
+    </xacro:macro>
+    <!-- Instantiate Wheels -->
+    <xacro:rearwheel prefix="left" x_reflect="-1" y_reflect="1"/>
+    <xacro:rearwheel prefix="right" x_reflect="-1" y_reflect="-1"/>
+    <xacro:steering_wheel prefix="left" x_reflect="1" y_reflect="1"/>
+    <xacro:steering_wheel prefix="right" x_reflect="1" y_reflect="-1"/>
+    <xacro:frontwheel prefix="left" x_reflect="1" y_reflect="1"/>
+    <xacro:frontwheel prefix="right" x_reflect="1" y_reflect="-1"/>
     <!-- Ackermann Steering Plugin -->
-    <plugin filename="gz-sim-ackermann-steering" name="gz::sim::systems::AckermannSteering">
-        <left_joint>rear_left_wheel_joint</left_joint>
-        <right_joint>rear_right_wheel_joint</right_joint>
-        <front_left_joint>front_left_steering_joint</front_left_joint>
-        <front_right_joint>front_right_steering_joint</front_right_joint>
-        <wheel_separation>0.287</wheel_separation>
-        <wheel_radius>${wheel_radius}</wheel_radius>
-        <max_linear_acceleration>0.033</max_linear_acceleration>
-        <topic>cmd_vel</topic>
-        <odom_topic>odom</odom_topic>
-        <frame_id>odom</frame_id>
-        <child_frame_id>base_footprint</child_frame_id>
-        <odom_publisher_frequency>30</odom_publisher_frequency>
-        <tf_topic>/tf</tf_topic>
+    <gazebo>
+        <plugin filename="libgz-sim-ackermann-steering.so" name="gz::sim::systems::AckermannSteering">
+            <left_joint>rear_left_wheel_joint</left_joint>
+            <right_joint>rear_right_wheel_joint</right_joint>
+            <front_left_joint>front_left_wheel_steering_joint</front_left_joint>
+            <front_right_joint>front_right_wheel_steering_joint</front_right_joint>
+            <wheel_separation>${base_width}</wheel_separation>
+            <wheel_radius>${wheel_radius}</wheel_radius>
+            <max_linear_acceleration>0.033</max_linear_acceleration>
+            <topic>cmd_vel</topic>
+            <odom_topic>odom</odom_topic>
+            <frame_id>odom</frame_id>
+            <child_frame_id>base_footprint</child_frame_id>
+            <odom_publisher_frequency>30</odom_publisher_frequency>
+            <tf_topic>/tf</tf_topic>
+        </plugin>
+    </gazebo>
+    <!-- Joint State Publisher -->
+    <plugin filename="gz-sim-joint-state-publisher-system"
+        name="gz::sim::systems::JointStatePublisher">
+        <topic>joint_states</topic>
+        <joint_name>rear_left_wheel_joint</joint_name>
+        <joint_name>rear_right_wheel_joint</joint_name>
+        <joint_name>front_left_wheel_steering_joint</joint_name>
+        <joint_name>front_right_wheel_steering_joint</joint_name>
     </plugin>
 </robot>

Commit message: test

File: isaac_ros-dev/src/agv_car_gazebo/urdf/car.xacro (robot description, xacro)
@@ -149,4 +149,21 @@
     </joint>
   </xacro:macro>
+  <plugin filename="gz-sim-ackermann-steering" name="gz::sim::systems::AckermannSteering">
+    <!-- Remove <ros> tag. -->
+    <!-- wheels -->
+    <left_joint>wheel_left_joint</left_joint>
+    <right_joint>wheel_right_joint</right_joint>
+    <!-- kinematics -->
+    <wheel_separation>0.287</wheel_separation>
+    <wheel_radius>0.033</wheel_radius> <!-- computed from <wheel_diameter> in the original plugin-->
+    <!-- limits -->
+    <max_linear_acceleration>0.033</max_linear_acceleration> <!-- computed from <max_linear_acceleration> in the original plugin-->
+    <topic>cmd_vel</topic> <!-- from <commant_topic> -->
+    <odom_topic>odom</odom_topic> <!-- from <odometry_topic> -->
+    <frame_id>odom</frame_id> <!-- from <odometry_frame> -->
+    <child_frame_id>base_footprint</child_frame_id> <!-- from <robot_base_frame> -->
+    <odom_publisher_frequency>30</odom_publisher_frequency> <!-- from <update_rate>-->
+    <tf_topic>/tf</tf_topic> <!-- Short topic name for tf output -->
+  </plugin>
   <!-- <link name="velodyne">
   <visual>

File: isaac_ros-dev/src/agv_car_gazebo/urdf/car1.urdf (robot description, URDF)
Before this commit: robot new_car, 6 links, 5 joints
Links:
- removed link front_left_steering_wheel
- removed link front_right_steering_wheel
- added link front_left_steering_wheel_link, mass 0.5; collision cylinder length=0.10000000 radius=0.029999999; visual cylinder length=0.1000000 radius=0.029999999
- added link front_left_wheel, mass 0.5; collision cylinder length=0.121 radius=0.191; visual cylinder length=0.121 radius=0.191
- added link front_right_steering_wheel_link, mass 0.5; collision cylinder length=0.10000000 radius=0.029999999; visual cylinder length=0.1000000 radius=0.029999999
- added link front_right_wheel, mass 0.5; collision cylinder length=0.121 radius=0.191; visual cylinder length=0.121 radius=0.191
Joints:
- removed joint front_left_steering_joint
- removed joint front_right_steering_joint
- added joint front_left_wheel_joint: type revolute, parent front_left_steering_wheel_link, child front_left_wheel, origin xyz=0 0 0 rpy=0 0 0, axis 0 0 1, limit lower=-0.698 upper=0.698 effort=1000.0 velocity=0.5
- added joint front_left_wheel_steering_joint: type revolute, parent base_link, child front_left_steering_wheel_link, origin xyz=0.756 0.46049999999999996 -0.123 rpy=0 0 0, axis 0 0 1, limit lower=-0.698 upper=0.698 effort=1000.0 velocity=0.5
- added joint front_right_wheel_joint: type revolute, parent front_right_steering_wheel_link, child front_right_wheel, origin xyz=0 0 0 rpy=0 0 0, axis 0 0 1, limit lower=-0.698 upper=0.698 effort=1000.0 velocity=0.5
- added joint front_right_wheel_steering_joint: type revolute, parent base_link, child front_right_steering_wheel_link, origin xyz=0.756 -0.46049999999999996 -0.123 rpy=0 0 0, axis 0 0 1, limit lower=-0.698 upper=0.698 effort=1000.0 velocity=0.5
