Commit message: Test

File: isaac_ros-dev/src/agv_car_gazebo/urdf/car.xacro (robot description, xacro)
@@ -41,23 +41,4 @@
       </collision>
       <xacro:box_inertia m="15" w="${base_width}" d="${base_length}" h="${base_height}"/>
-      <!-- Ackermann Steering Plugin -->
-      <gazebo>
-          <plugin filename="libgz-sim-ackermann-steering.so" name="gz::sim::systems::AckermannSteering">
-              <left_joint>rear_left_wheel_joint</left_joint>
-              <right_joint>rear_right_wheel_joint</right_joint>
-              <front_left_joint>front_left_wheel_steering_joint</front_left_joint>
-              <front_right_joint>front_right_wheel_steering_joint</front_right_joint>
-              <wheel_separation>0.287</wheel_separation>
-              <wheel_radius>${wheel_radius}</wheel_radius>
-              <max_linear_acceleration>0.033</max_linear_acceleration>
-              <topic>cmd_vel</topic>
-              <odom_topic>odom</odom_topic>
-              <frame_id>odom</frame_id>
-              <child_frame_id>base_footprint</child_frame_id>
-              <odom_publisher_frequency>30</odom_publisher_frequency>
-              <tf_topic>/tf</tf_topic>
-          </plugin>
-      </gazebo>
-  </link>
   <!-- Robot Footprint -->
   <link name="base_footprint"/>
@@ -241,4 +222,66 @@
     </inertial>
   </link> -->
+  <ros2_control name="GazeboSystem" type="system">
+    <hardware>
+      <plugin>gazebo_ros2_control/GazeboSystem</plugin>
+    </hardware>
+    <!-- Rear wheels -->
+    <joint name="rear_left_wheel_joint">
+      <command_interface name="velocity">
+        <param name="min">-10</param>
+        <param name="max">10</param>
+      </command_interface>
+      <state_interface name="position"/>
+      <state_interface name="velocity"/>
+    </joint>
+    <joint name="rear_right_wheel_joint">
+      <command_interface name="velocity">
+        <param name="min">-10</param>
+        <param name="max">10</param>
+      </command_interface>
+      <state_interface name="position"/>
+      <state_interface name="velocity"/>
+    </joint>
+    <!-- Steering wheel joints -->
+    <joint name="front_left_wheel_steering_joint">
+      <command_interface name="position">
+        <param name="min">-0.698</param>
+        <param name="max">0.698</param>
+      </command_interface>
+      <state_interface name="position"/>
+      <state_interface name="velocity"/>
+    </joint>
+    <joint name="front_right_wheel_steering_joint">
+      <command_interface name="position">
+        <param name="min">-0.698</param>
+        <param name="max">0.698</param>
+      </command_interface>
+      <state_interface name="position"/>
+      <state_interface name="velocity"/>
+    </joint>
+    <!-- Front wheels -->
+    <joint name="front_left_wheel_joint">
+      <command_interface name="velocity">
+        <param name="min">-10</param>
+        <param name="max">10</param>
+      </command_interface>
+      <state_interface name="position"/>
+      <state_interface name="velocity"/>
+    </joint>
+    <joint name="front_right_wheel_joint">
+      <command_interface name="velocity">
+        <param name="min">-10</param>
+        <param name="max">10</param>
+      </command_interface>
+      <state_interface name="position"/>
+      <state_interface name="velocity"/>
+    </joint>
+  </ros2_control>
+  <gazebo>
+    <!-- Joint state publisher -->
+    <plugin filename="libgazebo_ros2_control.so" name="gazebo_ros2_control">
+      <parameters>$(find wheeled_robot)/config/diff_drive_controller.yaml</parameters>
+    </plugin>
+  </gazebo>
   <xacro:rearwheel prefix="left" x_reflect="-1" y_reflect="1" />
   <xacro:rearwheel prefix="right" x_reflect="-1" y_reflect="-1" />
